File: Hardware/Fallout.kicad_sch (KiCad schematic)
At the start: 15 parts, among them J2 USB_C_Receptacle_USB2.0_14P, SW1 SW_Push, SW2 SW_Push, U1 ESP32-S3-WROOM-1, U2 AMS1117-3.3

Commit message: implemented Graphics pipeline
Parts:
- added J3: Conn_01x16, symbol Connector_Generic:Conn_01x16
Connections:
- net GND: now also J3.2 (Pin_2)
- net SCL: now also U1.10 (IO17); no longer U1.7 (IO7)
- net SDA: now also U1.11 (IO18); no longer U1.6 (IO6)
- net VCC: now also J3.1 (Pin_1), J3.7 (Pin_7)
- net LCD_D7: now reaches U1.12 (IO8)
- net LCD_D7: now also J3.15 (Pin_15)
- net LCD_D2: now reaches U1.15 (IO3)
- net LCD_D2: now also J3.10 (Pin_10)
- net LCD_RST: now reaches U1.17 (IO9)
- net LCD_RST: now also J3.3 (Pin_3)
- net LCD_CS: now reaches U1.18 (IO10)
- net LCD_CS: now also J3.4 (Pin_4)
- net LCD_RSDC: now reaches U1.19 (IO11)
- net LCD_RSDC: now also J3.5 (Pin_5)
- net LCD_WR: now reaches U1.20 (IO12)
- net LCD_WR: now also J3.6 (Pin_6)
- net LCD_D1: now reaches U1.38 (IO2)
- net LCD_D1: now also J3.9 (Pin_9)
- net LCD_D0: now reaches U1.39 (IO1)
- net LCD_D0: now also J3.8 (Pin_8)
- net LCD_D3: now reaches U1.4 (IO4)
- net LCD_D3: now also J3.11 (Pin_11)
- net LCD_D4: now reaches U1.5 (IO5)
- net LCD_D4: now also J3.12 (Pin_12)
- new net LCD_D5: J3.13 (Pin_13), U1.6 (IO6)
- new net LCD_D6: J3.14 (Pin_14), U1.7 (IO7)
Other:
- note added: "Screen"

Commit message: Gather hardware parts info
Parts:
- added J1: USB_A, symbol Connector:USB_A
- added Q1: IRF9540N, Package_TO_SOT_THT:TO-220-3_Vertical, symbol Transistor_FET:IRF9540N
- added Q2: 2N3904, Package_TO_SOT_THT:TO-92_Inline, symbol Transistor_BJT:2N3904
- added R7: 10k, symbol Device:R
- added R8: 1k~10k, symbol Device:R
- added SW3: SW_Push, symbol Switch:SW_Push
Connections:
- net D+: now also U1.14 (USB_D+), J1.3 (D+)
- net D-: now also U1.13 (USB_D-), J1.2 (D-)
- net GND: now also J1.4 (GND), J1.SH (Shield), Q2.1 (E), SW3.1
- net SCL: no longer U1.10 (IO17)
- net SDA: no longer U1.11 (IO18)
- net VBUS: now also Q1.3 (S), R7.2; no longer C3.2, U2.3 (VI)
- net POWER: now reaches U1.21 (IO13)
- net POWER: now also R8.1
- new net: Q1.1 (G), Q2.3 (C), R7.1, SW3.2
- new net: Q2.2 (B), R8.2
- new net VIN: C3.2, Q1.2 (D), U2.3 (VI)
Other:
- note added: "Power Button"
- note added: "USB-A Input"
- note added: "VBUS is the raw input from the USB-C VIN is the 5V input VCC is the 3V3 input"
